File: kicad_project/CargadorWalkieTalkie.kicad_sch (KiCad schematic)
At the start: 9 parts, among them J1 Screw_Terminal_01x02, J2 Screw_Terminal_01x02

Commit message: Agregando las capas y enrutamiento en las capas de la PCB
Signed-off-by: RoMadrigal <rmadrigalmontes@gmail.com>
Parts:
- D5: value 1N53xxB -> 1N5338B
Changed lines of the file:
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@@
 			)
 		)
-		(property "Value" "1N53xxB"
+		(property "Value" "1N5338B"
 			(at 168.91 83.8199 90)
 			(effects
